Commit message: added the endeffector link in the urdf

File: lbr_description/urdf/iiwa14/iiwa14.xacro (robot description, xacro)
@@ -4,4 +4,5 @@
     <!-- include the lbr iiwa macro -->
     <xacro:include filename="$(find lbr_description)/urdf/iiwa14/iiwa14_description.xacro" />
+    <xacro:include filename="$(find lbr_description)/urdf/iiwa14/beer_tool.xacro" />
     <xacro:arg name="robot_name" default="lbr" />
     <xacro:arg name="mode" default="true" />
@@ -14,4 +15,5 @@
         between world and link_0-->
     <joint name="world_joint" type="fixed">
+        <origin xyz="${0.61/2} 0.15 0.703" rpy="0.0 0.0 0.0"/>
         <parent link="world" />
         <child link="link_0" />
